File: Version_1/8_bit_Right_Rev_A.brd (EAGLE design)
At the start: 102.4 x 152.7 mm, 121 parts, among them IC1 74LS245N, IC10 7486N, IC11 7402N, IC12 74S08N, IC13 74LS173N, IC14 74LS173N, IC15 74LS245N, IC16 74LS139N, IC17 28C16AP, IC18 7476N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

Commit message: Fixed DRC problems
Routing:
- net N$44: track 55.2 -> 51.2 mm
- net N$48: track 16.1 -> 12.8 mm
- net VCC: track 687.9 -> 684.9 mm
- net GND: track 988.5 -> 985.6 mm
- net N$88: track 68.5 -> 66.4 mm
- net N$94: track 59.0 -> 57.7 mm
- net N_EO: track 123.5 -> 122.2 mm
- net SU: track 357.9 -> 356.9 mm
- net N$87: track 69.9 -> 68.9 mm
