File: Version_1/8_bit_Middle_Rev_A.brd (EAGLE design)
At the start: 62.2 x 163.1 mm, 42 parts

Commit message: Trash image on the other side
Parts:
- moved U$2 11.4 mm to (35.7, 2.82), flipped to the bottom
Changed lines of the file:
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@@
 </element>
 <element name="U$1" library="Logos" package="SOLAIRE" value="" x="1.2446" y="105.9942" smashed="yes"/>
-<element name="U$2" library="logo" library_urn="urn:adsk.eagle:library:264" package="MUELLTONNE" value="" x="24.2824" y="2.8194" smashed="yes"/>
+<element name="U$2" library="logo" library_urn="urn:adsk.eagle:library:264" package="MUELLTONNE" value="" x="35.6616" y="2.8194" smashed="yes" rot="MR0"/>
 </elements>
 <signals>
